Commit message: updated robot gates and changed costmap

File: spherebot_description/urdf/spherebot.urdf (robot description, URDF)
Before this commit: robot u_shaped_collector_v2, 10 links, 9 joints
Links:
- link right_gate: geometry collision box size=0.02 0.10 0.18; visual box size=0.02 0.10 0.18

File: spherebot_description/urdf/spherebot.urdf.xacro (robot description, xacro)
@@ -29,9 +29,9 @@
   <!-- Gate Dimensions -->
   <xacro:property name="gate_thick" value="0.02"/>
-  <xacro:property name="gate_len" value="0.18"/>
+  <xacro:property name="gate_len" value="0.09"/>
   <xacro:property name="gate_height" value="0.18"/>
   <xacro:property name="gate_mass" value="0.1"/>
   <xacro:property name="gate_x_mount" value="0.4"/>
-  <xacro:property name="gate_y_mount" value="0.25"/>
+  <xacro:property name="gate_y_mount" value="0.205"/>
   <xacro:property name="gate_travel" value="0.25"/>
   <!-- Colors -->
