Commit message: spherebot control (twist + gate)

File: spherebot_description/urdf/spherebot.urdf.xacro (robot description, xacro)
@@ -13,5 +13,5 @@
   <xacro:property name="arm_thick" value="0.05"/>
   <xacro:property name="arm_height" value="0.2"/>
-  <xacro:property name="arm_y_offset" value="0.185"/> <!-- Distance from center to arm center -->
+  <xacro:property name="arm_y_offset" value="0.185"/>
   <xacro:property name="arm_x_offset" value="0.225"/>
   <!-- Wheel Dimensions -->
@@ -33,5 +33,5 @@
   <xacro:property name="gate_mass" value="0.1"/>
   <xacro:property name="gate_x_mount" value="0.4"/>
-  <xacro:property name="gate_y_mount" value="0.25"/> <!-- Adjusted offset per previous request -->
+  <xacro:property name="gate_y_mount" value="0.25"/>
   <xacro:property name="gate_travel" value="0.25"/>
   <!-- Colors -->
@@ -40,4 +40,7 @@
   <material name="red"><color rgba="0.8 0 0 1"/></material>
   <material name="silver"><color rgba="0.7 0.7 0.7 1"/></material>
+  <!-- [NEW] ARGUMENT FOR CONTROLLER CONFIG -->
+  <!-- This allows the launch file to pass in the path to the yaml file -->
+  <xacro:arg name="config_file" default="$(find spherebot_control)/config/controllers.yaml" />
   <!-- ======================================================================= -->
   <!--                           INERTIA MACROS                                -->
@@ -82,8 +85,15 @@
       <xacro:cylinder_inertia m="${wheel_mass}" r="${wheel_radius}" h="${wheel_width}"/>
     </link>
+    <gazebo reference="${prefix}_wheel">
+      <mu1>1.0</mu1>
+      <mu2>1.0</mu2>
+      <kp>1000000.0</kp>
+      <kd>100.0</kd>
+      <minDepth>0.001</minDepth>
+      <maxVel>1.0</maxVel>
+    </gazebo>
     <joint name="${prefix}_wheel_joint" type="continuous">
       <parent link="base_link"/>
       <child link="${prefix}_wheel"/>
-      <!-- reflect is 1 for left, -1 for right -->
       <origin xyz="${wheel_x_offset} ${reflect * wheel_y_offset} ${wheel_z_offset}" rpy="-1.5708 0 0"/>
       <axis xyz="0 0 1"/>
@@ -109,19 +119,8 @@
       <limit lower="${lower_lim}" upper="${upper_lim}" effort="10" velocity="0.5"/>
     </joint>
-    <!-- Individual controller plugin for this gate -->
-    <gazebo>
-      <plugin filename="gz-sim-joint-position-controller-system" name="gz::sim::systems::JointPositionController">
-        <joint_name>${prefix}_gate_joint</joint_name>
-        <p_gain>10</p_gain>
-        <i_gain>0.1</i_gain>
-        <d_gain>0.1</d_gain>
-        <topic>gate/${prefix}/cmd_pos</topic>
-      </plugin>
-    </gazebo>
   </xacro:macro>
   <!-- ======================================================================= -->
   <!--                           MAIN ROBOT STRUCTURE                          -->
   <!-- ======================================================================= -->
-  <!-- Base Footprint (World Ground Projection) -->
   <link name="base_footprint"/>
   <joint name="base_joint" type="fixed">
@@ -130,7 +129,6 @@
     <origin xyz="0 0 0.14" rpy="0 0 0"/>
   </joint>
-  <!-- Base Link (Complex Shape: Center + 2 Arms) -->
   <link name="base_link">
-    <!-- 1. Center Body -->
+    <!-- Center Body -->
     <visual>
       <origin xyz="0 0 0"/>
@@ -142,5 +140,5 @@
       <geometry><box size="${base_len} ${base_width} ${base_height}"/></geometry>
     </collision>
-    <!-- 2. Left Arm -->
+    <!-- Left Arm -->
     <visual>
       <origin xyz="${arm_x_offset} ${arm_y_offset} 0"/>
@@ -152,5 +150,5 @@
       <geometry><box size="${arm_len} ${arm_thick} ${arm_height}"/></geometry>
     </collision>
-    <!-- 3. Right Arm -->
+    <!-- Right Arm -->
     <visual>
       <origin xyz="${arm_x_offset} -${arm_y_offset} 0"/>
@@ -162,11 +160,8 @@
       <geometry><box size="${arm_len} ${arm_thick} ${arm_height}"/></geometry>
     </collision>
-    <!-- Combined Inertia (Simplified as one big box for stability) -->
     <xacro:box_inertia m="${base_mass}" l="0.4" w="0.42" h="0.2"/>
   </link>
-  <!-- Instantiate Wheels -->
   <xacro:wheel prefix="left" reflect="1"/>
   <xacro:wheel prefix="right" reflect="-1"/>
-  <!-- Instantiate Caster Wheel -->
   <link name="caster_wheel">
     <visual>
@@ -188,11 +183,64 @@
     <material>Gazebo/Silver</material>
   </gazebo>
-  <!-- Instantiate Sliding Gates -->
   <xacro:sliding_gate prefix="left" y_pos="${gate_y_mount}" lower_lim="-${gate_travel}" upper_lim="0"/>
   <xacro:sliding_gate prefix="right" y_pos="-${gate_y_mount}" lower_lim="0" upper_lim="${gate_travel}"/>
   <!-- ======================================================================= -->
+  <!--                       ROS 2 CONTROL INTERFACE                           -->
+  <!-- ======================================================================= -->
+  <ros2_control name="GazeboSimSystem" type="system">
+    <hardware>
+      <plugin>gz_ros2_control/GazeboSimSystem</plugin>
+    </hardware>
+    <!-- Differential Drive Wheels -->
+    <joint name="left_wheel_joint">
+      <command_interface name="velocity">
+        <param name="min">-10</param>
+        <param name="max">10</param>
+      </command_interface>
+      <state_interface name="velocity"/>
+      <state_interface name="position"/>
+    </joint>
+    <joint name="right_wheel_joint">
+      <command_interface name="velocity">
+        <param name="min">-10</param>
+        <param name="max">10</param>
+      </command_interface>
+      <state_interface name="velocity"/>
+      <state_interface name="position"/>
+    </joint>
+    <!-- Sliding Gates -->
+    <joint name="left_gate_joint">
+      <command_interface name="position">
+        <param name="min">-${gate_travel}</param>
+        <param name="max">0</param>
+      </command_interface>
+      <state_interface name="position"/>
+      <state_interface name="velocity"/>
+    </joint>
+    <joint name="right_gate_joint">
+      <command_interface name="position">
+        <param name="min">0</param>
+        <param name="max">${gate_travel}</param>
+      </command_interface>
+      <state_interface name="position"/>
+      <state_interface name="velocity"/>
+    </joint>
+  </ros2_control>
+  <!-- ======================================================================= -->
+  <!--                           GAZEBO PLUGINS                                -->
+  <!-- ======================================================================= -->
+  <gazebo>
+    <!-- [UPDATED] ROS 2 Control Bridge -->
+    <!-- It now uses the 'config_file' argument passed from the launch file -->
+    <plugin filename="gz_ros2_control-system" name="gz_ros2_control::GazeboSimROS2ControlPlugin">
+      <parameters>$(arg config_file)</parameters>
+    </plugin>
+    <!-- Sensors remain unchanged -->
+    <plugin filename="gz-sim-imu-system" name="gz::sim::systems::Imu">
+    </plugin>
+  </gazebo>
+  <!-- ======================================================================= -->
   <!--                           SENSORS                                       -->
   <!-- ======================================================================= -->
-  <!-- LiDAR -->
   <link name="lidar_link">
     <visual>
@@ -234,5 +282,4 @@
     </sensor>
   </gazebo>
-  <!-- Camera -->
   <link name="camera_link">
     <visual>
@@ -240,5 +287,4 @@
       <material name="red"/>
     </visual>
-    <!-- Camera is lightweight, negligible inertia/collision for simulation simplicity usually -->
   </link>
   <joint name="camera_joint" type="fixed">
@@ -273,5 +319,4 @@
     </sensor>
   </gazebo>
-  <!-- IMU -->
   <link name="imu_link">
     <inertial>
@@ -305,37 +350,3 @@
     </sensor>
   </gazebo>
-  <!-- ======================================================================= -->
-  <!--                           GAZEBO PLUGINS                                -->
-  <!-- ======================================================================= -->
-  <gazebo>
-    <!-- Joint State Publisher (Publishes /joint_states) -->
-    <plugin filename="gz-sim-joint-state-publisher-system" name="gz::sim::systems::JointStatePublisher">
-      <topic>joint_states</topic>
-    </plugin>
-    <!-- Differential Drive Controller -->
-    <plugin filename="gz-sim-diff-drive-system" name="gz::sim::systems::DiffDrive">
-      <left_joint>left_wheel_joint</left_joint>
-      <right_joint>right_wheel_joint</right_joint>
-      <wheel_separation>0.47</wheel_separation>
-      <wheel_radius>${wheel_radius}</wheel_radius>
-      <odom_publish_frequency>20</odom_publish_frequency>
-      <topic>cmd_vel</topic>
-      <odom_topic>odom</odom_topic>
-      <tf_topic>tf</tf_topic>
-      <frame_id>odom</frame_id>
-      <child_frame_id>base_footprint</child_frame_id>
-    </plugin>
-    <!-- Odometry Publisher (Ground Truth) -->
-    <plugin filename="gz-sim-odometry-publisher-system" name="gz::sim::systems::OdometryPublisher">
-      <odom_frame>odom</odom_frame>
-      <robot_base_frame>base_footprint</robot_base_frame>
-      <odom_publish_frequency>50</odom_publish_frequency>
-      <odom_topic>odom</odom_topic>
-      <tf_topic>tf</tf_topic>
-      <dimensions>3</dimensions>
-    </plugin>
-    <!-- IMU System -->
-    <plugin filename="gz-sim-imu-system" name="gz::sim::systems::Imu">
-    </plugin>
-  </gazebo>
 </robot>

Commit message: spawn spheres

File: spherebot_description/urdf/spherebot.urdf.xacro (robot description, xacro)
@@ -29,9 +29,9 @@
   <!-- Gate Dimensions -->
   <xacro:property name="gate_thick" value="0.02"/>
-  <xacro:property name="gate_len" value="0.09"/>
+  <xacro:property name="gate_len" value="0.18"/>
   <xacro:property name="gate_height" value="0.18"/>
   <xacro:property name="gate_mass" value="0.1"/>
   <xacro:property name="gate_x_mount" value="0.4"/>
-  <xacro:property name="gate_y_mount" value="0.205"/>
+  <xacro:property name="gate_y_mount" value="0.25"/>
   <xacro:property name="gate_travel" value="0.25"/>
   <!-- Colors -->

Commit message: updated robot to catch big blue sphere

File: spherebot_description/urdf/spherebot.urdf.xacro (robot description, xacro)
@@ -6,19 +6,19 @@
   <!-- Base Dimensions -->
   <xacro:property name="base_len" value="0.1"/>
-  <xacro:property name="base_width" value="0.42"/>
+  <xacro:property name="base_width" value="0.63"/>
   <xacro:property name="base_height" value="0.2"/>
   <xacro:property name="base_mass" value="10.0"/>
   <!-- U-Arm Dimensions -->
-  <xacro:property name="arm_len" value="0.35"/>
-  <xacro:property name="arm_thick" value="0.05"/>
+  <xacro:property name="arm_len" value="0.6"/>
+  <xacro:property name="arm_thick" value="0.02"/>
   <xacro:property name="arm_height" value="0.2"/>
-  <xacro:property name="arm_y_offset" value="0.185"/>
-  <xacro:property name="arm_x_offset" value="0.225"/>
+  <xacro:property name="arm_y_offset" value="0.31"/>
+  <xacro:property name="arm_x_offset" value="0.250"/>
   <!-- Wheel Dimensions -->
   <xacro:property name="wheel_radius" value="0.06"/>
   <xacro:property name="wheel_width" value="0.04"/>
   <xacro:property name="wheel_mass" value="0.5"/>
-  <xacro:property name="wheel_x_offset" value="0.3"/>
-  <xacro:property name="wheel_y_offset" value="0.235"/>
+  <xacro:property name="wheel_x_offset" value="0.45"/>
+  <xacro:property name="wheel_y_offset" value="0.335"/>
   <xacro:property name="wheel_z_offset" value="-0.08"/>
   <!-- Caster Dimensions -->
@@ -29,5 +29,5 @@
   <!-- Gate Dimensions -->
   <xacro:property name="gate_thick" value="0.02"/>
-  <xacro:property name="gate_len" value="0.18"/>
+  <xacro:property name="gate_len" value="0.30"/>
   <xacro:property name="gate_height" value="0.18"/>
   <xacro:property name="gate_mass" value="0.1"/>
@@ -100,24 +100,37 @@
     </joint>
   </xacro:macro>
-  <!-- Sliding Gate Macro -->
-  <xacro:macro name="sliding_gate" params="prefix y_pos lower_lim upper_lim">
-    <link name="${prefix}_gate">
-      <visual>
-        <geometry><box size="${gate_thick} ${gate_len} ${gate_height}"/></geometry>
-        <material name="red"/>
-      </visual>
-      <collision>
-        <geometry><box size="${gate_thick} ${gate_len} ${gate_height}"/></geometry>
-      </collision>
-      <xacro:box_inertia m="${gate_mass}" l="${gate_thick}" w="${gate_len}" h="${gate_height}"/>
-    </link>
-    <joint name="${prefix}_gate_joint" type="prismatic">
-      <parent link="base_link"/>
-      <child link="${prefix}_gate"/>
-      <origin xyz="${gate_x_mount} ${y_pos} 0" rpy="0 0 0"/>
-      <axis xyz="0 1 0"/>
-      <limit lower="${lower_lim}" upper="${upper_lim}" effort="10" velocity="0.5"/>
-    </joint>
-  </xacro:macro>
+<xacro:macro name="revolute_gate" params="prefix y_sign axis_sign">
+  <link name="${prefix}_gate">
+    <visual>
+      <!-- Gate extends forward from hinge -->
+      <origin xyz="${gate_len/2} 0 0"/>
+      <geometry>
+        <box size="${gate_len} ${gate_thick} ${gate_height}"/>
+      </geometry>
+      <material name="red"/>
+    </visual>
+    <collision>
+      <origin xyz="${gate_len/2} 0 0"/>
+      <geometry>
+        <box size="${gate_len} ${gate_thick} ${gate_height}"/>
+      </geometry>
+    </collision>
+    <xacro:box_inertia
+      m="${gate_mass}"
+      l="${gate_len}"
+      w="${gate_thick}"
+      h="${gate_height}"/>
+  </link>
+  <joint name="${prefix}_gate_joint" type="revolute">
+  <parent link="base_link"/>
+  <child link="${prefix}_gate"/>
+  <origin
+    xyz="${arm_x_offset + arm_len/2} ${y_sign * arm_y_offset} 0"
+    rpy="0 0 0"/>
+  <axis xyz="0 0 ${axis_sign}"/>
+  <limit lower="0.0" upper="1.57" effort="15.0" velocity="2.0"/>
+  <dynamics damping="0.5" friction="0.3"/>
+</joint>
+</xacro:macro>
   <!-- ======================================================================= -->
   <!--                           MAIN ROBOT STRUCTURE                          -->
@@ -183,6 +196,6 @@
     <material>Gazebo/Silver</material>
   </gazebo>
-  <xacro:sliding_gate prefix="left" y_pos="${gate_y_mount}" lower_lim="-${gate_travel}" upper_lim="0"/>
-  <xacro:sliding_gate prefix="right" y_pos="-${gate_y_mount}" lower_lim="0" upper_lim="${gate_travel}"/>
+  <xacro:revolute_gate prefix="left"  y_sign="1"  axis_sign="-1"/>
+  <xacro:revolute_gate prefix="right" y_sign="-1" axis_sign="1"/>
   <!-- ======================================================================= -->
   <!--                       ROS 2 CONTROL INTERFACE                           -->
@@ -209,21 +222,20 @@
       <state_interface name="position"/>
     </joint>
-    <!-- Sliding Gates -->
     <joint name="left_gate_joint">
-      <command_interface name="position">
-        <param name="min">-${gate_travel}</param>
-        <param name="max">0</param>
-      </command_interface>
-      <state_interface name="position"/>
-      <state_interface name="velocity"/>
-    </joint>
-    <joint name="right_gate_joint">
-      <command_interface name="position">
-        <param name="min">0</param>
-        <param name="max">${gate_travel}</param>
-      </command_interface>
-      <state_interface name="position"/>
-      <state_interface name="velocity"/>
-    </joint>
+  <command_interface name="position">
+    <param name="min">0.0</param>
+    <param name="max">1.57</param>
+  </command_interface>
+  <state_interface name="position"/>
+  <state_interface name="velocity"/>
+</joint>
+<joint name="right_gate_joint">
+  <command_interface name="position">
+    <param name="min">0.0</param>
+    <param name="max">1.57</param>
+  </command_interface>
+  <state_interface name="position"/>
+  <state_interface name="velocity"/>
+</joint>
   </ros2_control>
   <!-- ======================================================================= -->

Commit message: lidar on increased height

File: spherebot_description/urdf/spherebot.urdf.xacro (robot description, xacro)
@@ -35,4 +35,8 @@
   <xacro:property name="gate_y_mount" value="0.25"/>
   <xacro:property name="gate_travel" value="0.25"/>
+  <!-- Lidar Stand Dimensions -->
+  <xacro:property name="lidar_stand_height" value="0.4"/>
+  <xacro:property name="lidar_stand_radius" value="0.02"/>
+  <xacro:property name="lidar_stand_mass" value="0.3"/>
   <!-- Colors -->
   <material name="blue"><color rgba="0 0 0.8 1"/></material>
@@ -258,4 +262,30 @@
   <!--                           SENSORS                                       -->
   <!-- ======================================================================= -->
+  <link name="lidar_stand_link">
+  <visual>
+    <!-- Center of cylinder is half its height -->
+    <origin xyz="0 0 ${lidar_stand_height/2}" rpy="0 0 0"/>
+    <geometry>
+      <cylinder length="${lidar_stand_height}" radius="${lidar_stand_radius}"/>
+    </geometry>
+    <material name="silver"/>
+  </visual>
+  <collision>
+    <origin xyz="0 0 ${lidar_stand_height/2}" rpy="0 0 0"/>
+    <geometry>
+      <cylinder length="${lidar_stand_height}" radius="${lidar_stand_radius}"/>
+    </geometry>
+  </collision>
+  <xacro:cylinder_inertia
+    m="${lidar_stand_mass}"
+    r="${lidar_stand_radius}"
+    h="${lidar_stand_height}"/>
+</link>
+<joint name="lidar_stand_joint" type="fixed">
+  <parent link="base_link"/>
+  <child link="lidar_stand_link"/>
+  <origin xyz="-0.01 0 0.1" rpy="0 0 0"/>
+</joint>
+  <!-- Lidar -->
   <link name="lidar_link">
     <visual>
@@ -269,8 +299,8 @@
   </link>
   <joint name="lidar_joint" type="fixed">
-    <parent link="base_link"/>
-    <child link="lidar_link"/>
-    <origin xyz="-0.01 0 0.12" rpy="0 0 0"/>
-  </joint>
+  <parent link="lidar_stand_link"/>
+  <child link="lidar_link"/>
+  <origin xyz="0 0 ${lidar_stand_height + 0.02}" rpy="0 0 0"/>
+</joint>
   <gazebo reference="lidar_link">
     <sensor name="lidar" type="gpu_lidar">

Commit message: basic opencv detection for red ball with approach

File: spherebot_description/urdf/spherebot.urdf.xacro (robot description, xacro)
@@ -44,4 +44,5 @@
   <material name="red"><color rgba="0.8 0 0 1"/></material>
   <material name="silver"><color rgba="0.7 0.7 0.7 1"/></material>
+  <material name="gray"><color rgba="0.5 0.5 0.5 1"/></material>
   <!-- [NEW] ARGUMENT FOR CONTROLLER CONFIG -->
   <!-- This allows the launch file to pass in the path to the yaml file -->
@@ -112,5 +113,5 @@
         <box size="${gate_len} ${gate_thick} ${gate_height}"/>
       </geometry>
-      <material name="red"/>
+      <material name="gray"/>
     </visual>
     <collision>
@@ -126,4 +127,7 @@
       h="${gate_height}"/>
   </link>
+  <gazebo reference="${prefix}_gate">
+  <material>Gazebo/Grey</material>
+</gazebo>
   <joint name="${prefix}_gate_joint" type="revolute">
   <parent link="base_link"/>

Commit message: partial working blue ball chase with obstacle avoidance

File: spherebot_description/urdf/spherebot.urdf.xacro (robot description, xacro)
@@ -17,8 +17,8 @@
   <!-- Wheel Dimensions -->
   <xacro:property name="wheel_radius" value="0.06"/>
-  <xacro:property name="wheel_width" value="0.04"/>
+  <xacro:property name="wheel_width" value="0.02"/>
   <xacro:property name="wheel_mass" value="0.5"/>
   <xacro:property name="wheel_x_offset" value="0.45"/>
-  <xacro:property name="wheel_y_offset" value="0.335"/>
+  <xacro:property name="wheel_y_offset" value="0.310"/>
   <xacro:property name="wheel_z_offset" value="-0.08"/>
   <!-- Caster Dimensions -->
